Commit message: add a gimbal to the generic camera

File: hector_sensors_description/urdf/generic_camera.urdf.xacro (robot description, xacro)
@@ -7,8 +7,24 @@
     <property name="M_PI" value="3.1415926535897931" />
     <xacro:macro name="generic_camera" params="name parent *origin ros_topic cam_info_topic update_rate res_x res_y image_format hfov">
-      <joint name="${name}_joint" type="fixed">
+      <joint name="${name}_roll" type="continuous">
         <insert_block name="origin" />
         <parent link="${parent}"/>
+        <child link="${name}_interm_link"/>
+	<axis xyz="1 0 0" />
+	<limit effort="0.1" lower="${-M_PI/4}" upper="${M_PI/4}" velocity="0.2" />
+      </joint>
+      <link name="${name}_interm_link" >
+	<inertial>
+	  <mass value="0.0001" />
+	  <origin xyz="0 0 0" rpy="0 0 0" />
+          <inertia ixx="0.00001" ixy="0" ixz="0" iyy="0.00001" iyz="0" izz="0.00001" />
+	</inertial>
+      </link>
+      <joint name="${name}_pitch" type="continuous">
+        <insert_block name="origin" />
+        <parent link="${name}_interm_link"/>
         <child link="${name}_link"/>
+	<axis xyz="0 1 0" />
+	<limit effort="0.1" lower="${-M_PI/4}" upper="${M_PI/4}" velocity="0.2" />
       </joint>
       <link name="${name}_link">
@@ -24,6 +40,6 @@
           </geometry>
 	  <material name="Blue">
-      <color rgba="0.0 0.0 0.8 1"/>
-    </material>
+	    <color rgba="0.0 0.0 0.8 1"/>
+	  </material>
         </visual>
         <collision>

Commit message: make this camera match a gopro and fix the joint types to revolute

File: hector_sensors_description/urdf/generic_camera.urdf.xacro (robot description, xacro)
@@ -7,5 +7,5 @@
     <property name="M_PI" value="3.1415926535897931" />
     <xacro:macro name="generic_camera" params="name parent *origin ros_topic cam_info_topic update_rate res_x res_y image_format hfov">
-      <joint name="${name}_roll" type="continuous">
+      <joint name="${name}_roll" type="revolute">
         <insert_block name="origin" />
         <parent link="${parent}"/>
@@ -16,10 +16,11 @@
       <link name="${name}_interm_link" >
 	<inertial>
-	  <mass value="0.0001" />
+	  <mass value="0.010" />
 	  <origin xyz="0 0 0" rpy="0 0 0" />
-          <inertia ixx="0.00001" ixy="0" ixz="0" iyy="0.00001" iyz="0" izz="0.00001" />
+	  <!-- assume a sphere of r = 1cm - 2/5 * mr^2 = 4e-7 -->
+          <inertia ixx="4e-7" ixy="0" ixz="0" iyy="4e-7" iyz="0" izz="4e-7" />
 	</inertial>
       </link>
-      <joint name="${name}_pitch" type="continuous">
+      <joint name="${name}_pitch" type="revolute">
         <insert_block name="origin" />
         <parent link="${name}_interm_link"/>
@@ -30,15 +31,21 @@
       <link name="${name}_link">
         <inertial>
-          <mass value="0.001" />
+          <mass value="0.172" />
           <origin xyz="0 0 0" rpy="0 0 0" />
-          <inertia ixx="0.0001" ixy="0" ixz="0" iyy="0.0001" iyz="0" izz="0.0001" />
+	  <!-- x = depth
+	       y = width
+	       z = height
+	  solid cube = 1/12 * m( h^2 + w^2 ) - 0.000077
+	                    1/12 * m( h^2 + d^2 ) - 0.000037
+			    1/12 * m( w^2 + d^2 ) - 0.000065 -->
+          <inertia ixx="0.000077" ixy="0" ixz="0" iyy="0.00037" iyz="0" izz="0.000065" />
         </inertial>
         <visual>
           <origin xyz="0 0 0" rpy="0 0 0" />
           <geometry>
-            <box size="0.01 0.01 0.01" />
+            <box size="0.030 0.060 0.041" />
           </geometry>
-	  <material name="Blue">
-	    <color rgba="0.0 0.0 0.8 1"/>
+	  <material name="Grey">
+	    <color rgba="0.5 0.5 0.5 1"/>
 	  </material>
         </visual>
@@ -46,5 +53,5 @@
           <origin xyz="0 0 0" rpy="0 0 0" />
           <geometry>
-            <box size="0.01 0.01 0.01" />
+            <box size="0.030 0.060 0.041" />
           </geometry>
         </collision>

Commit message: change pr2/blue to white

File: hector_sensors_description/urdf/generic_camera.urdf.xacro (robot description, xacro)
@@ -102,5 +102,5 @@
       </sensor:camera>
       <turnGravityOff>true</turnGravityOff>
-      <material>PR2/Blue</material>
+      <material>white</material>
     </gazebo>
     </xacro:macro>

Commit message: Revert "make this camera match a gopro and fix the joint types to revolute"
This reverts commit b3ac9a2eed0fa82efe1162d53649a37c5e698350.

File: hector_sensors_description/urdf/generic_camera.urdf.xacro (robot description, xacro)
@@ -7,5 +7,5 @@
     <property name="M_PI" value="3.1415926535897931" />
     <xacro:macro name="generic_camera" params="name parent *origin ros_topic cam_info_topic update_rate res_x res_y image_format hfov">
-      <joint name="${name}_roll" type="revolute">
+      <joint name="${name}_roll" type="continuous">
         <insert_block name="origin" />
         <parent link="${parent}"/>
@@ -16,11 +16,10 @@
       <link name="${name}_interm_link" >
 	<inertial>
-	  <mass value="0.010" />
+	  <mass value="0.0001" />
 	  <origin xyz="0 0 0" rpy="0 0 0" />
-	  <!-- assume a sphere of r = 1cm - 2/5 * mr^2 = 4e-7 -->
-          <inertia ixx="4e-7" ixy="0" ixz="0" iyy="4e-7" iyz="0" izz="4e-7" />
+          <inertia ixx="0.00001" ixy="0" ixz="0" iyy="0.00001" iyz="0" izz="0.00001" />
 	</inertial>
       </link>
-      <joint name="${name}_pitch" type="revolute">
+      <joint name="${name}_pitch" type="continuous">
         <insert_block name="origin" />
         <parent link="${name}_interm_link"/>
@@ -31,21 +30,15 @@
       <link name="${name}_link">
         <inertial>
-          <mass value="0.172" />
+          <mass value="0.001" />
           <origin xyz="0 0 0" rpy="0 0 0" />
-	  <!-- x = depth
-	       y = width
-	       z = height
-	  solid cube = 1/12 * m( h^2 + w^2 ) - 0.000077
-	                    1/12 * m( h^2 + d^2 ) - 0.000037
-			    1/12 * m( w^2 + d^2 ) - 0.000065 -->
-          <inertia ixx="0.000077" ixy="0" ixz="0" iyy="0.00037" iyz="0" izz="0.000065" />
+          <inertia ixx="0.0001" ixy="0" ixz="0" iyy="0.0001" iyz="0" izz="0.0001" />
         </inertial>
         <visual>
           <origin xyz="0 0 0" rpy="0 0 0" />
           <geometry>
-            <box size="0.030 0.060 0.041" />
+            <box size="0.01 0.01 0.01" />
           </geometry>
-	  <material name="Grey">
-	    <color rgba="0.5 0.5 0.5 1"/>
+	  <material name="Blue">
+	    <color rgba="0.0 0.0 0.8 1"/>
 	  </material>
         </visual>
@@ -53,5 +46,5 @@
           <origin xyz="0 0 0" rpy="0 0 0" />
           <geometry>
-            <box size="0.030 0.060 0.041" />
+            <box size="0.01 0.01 0.01" />
           </geometry>
         </collision>

Commit message: correct color

File: hector_sensors_description/urdf/generic_camera.urdf.xacro (robot description, xacro)
@@ -95,5 +95,7 @@
       </sensor:camera>
       <turnGravityOff>true</turnGravityOff>
-      <material>white</material>
+      <material>
+	<color rgba="1.0 1.0 1.0 1.0"/>
+      </material>
     </gazebo>
     </xacro:macro>

Commit message: remove material

File: hector_sensors_description/urdf/generic_camera.urdf.xacro (robot description, xacro)
@@ -95,7 +95,4 @@
       </sensor:camera>
       <turnGravityOff>true</turnGravityOff>
-      <material>
-	<color rgba="1.0 1.0 1.0 1.0"/>
-      </material>
     </gazebo>
     </xacro:macro>
